Commit message: feat: add 3-LiDAR sensor stack (Hesai XT32 + dual RoboSense RSE1)
- Add HesaiLidar_ROS_2.0 submodule (Hesai XT32, 192.168.1.201)
- Add rslidar_sdk + rslidar_msg submodules (RoboSense RSE1 Left/Right)
- Add pylon_ros2_camera submodule with Jazzy compat patches
- Add raptorlift_camera package (Basler camera launch)
- Update URDF: lidar_rslidar_left_link + lidar_rslidar_right_link
- Add docs/lidar_setting.md with network, port, TF documentation
- Update setup_env.bash with LiDAR launch commands

File: src/raptorlift_description/urdf/raptorlift.urdf (robot description, URDF)
Before this commit: robot raptorlift, 11 links, 10 joints
Links:
- added link lidar_rslidar_left_link, mass 0.3; collision cylinder length=0.055 radius=0.052; visual cylinder length=0.055 radius=0.052
- added link lidar_rslidar_right_link, mass 0.3; collision cylinder length=0.055 radius=0.052; visual cylinder length=0.055 radius=0.052
Joints:
- added joint lidar_rslidar_left_joint: type fixed, parent base_link, child lidar_rslidar_left_link, origin xyz=0.0 0.35 0.55 rpy=0 0 0
- added joint lidar_rslidar_right_joint: type fixed, parent base_link, child lidar_rslidar_right_link, origin xyz=0.0 -0.35 0.55 rpy=0 0 0

Commit message: SP01_Slam

File: src/raptorlift_description/urdf/raptorlift.urdf (robot description, URDF)
Before this commit: robot raptorlift, 13 links, 12 joints
Links:
- removed link lidar_rslidar_left_link
- removed link lidar_rslidar_right_link
- added link lidar_rslidar_back_link, mass 0.3; collision cylinder length=0.055 radius=0.052; visual cylinder length=0.055 radius=0.052
- added link lidar_rslidar_front_link, mass 0.3; collision cylinder length=0.055 radius=0.052; visual cylinder length=0.055 radius=0.052
Joints:
- removed joint lidar_rslidar_left_joint
- removed joint lidar_rslidar_right_joint
- added joint lidar_rslidar_back_joint: type fixed, parent base_link, child lidar_rslidar_back_link, origin xyz=-0.55 0.0 0.55 rpy=0 0 0
- added joint lidar_rslidar_front_joint: type fixed, parent base_link, child lidar_rslidar_front_link, origin xyz=0.55 0.0 0.55 rpy=0 0 0

Commit message: fix: rear-steer Ackermann steering direction + comprehensive improvements
- Fix steering inversion: negate steering angle at hardware boundary for
  rear-steer so +angular.z = LEFT turn (ROS convention)
- Unify PID controller: single canonical implementation in
  raptorlift_hardware_bridge, namespace alias in raptorlift_hardware
- VirtualPLC physics: replace hardcoded gains with proper inertia/damping
  model matching raptorlift_hardware.cpp, wire YAML simulation params
- Nav2: adjust costmap footprint to actual chassis size (1.1x0.8m),
  remove physically impossible spin behavior for Ackermann
- Teleop: scale angular velocity proportionally with gear (low gear =
  lower omega limit, matching steering angle constraints)
- Fix stale dt in read_from_hardware, e-stop steering reset,
  VirtualPLC steering snap-back at angle limits

File: src/raptorlift_description/urdf/raptorlift.urdf (robot description, URDF)
Before this commit: robot raptorlift, 13 links, 12 joints
Joints:
- joint rear_right_steering_joint: origin xyz=-0.52235 -0.355 -0.0705 rpy=0 0 3.1416 -> xyz=-0.52235 -0.355 -0.0705 rpy=0 0 0
